Commit message: Add files via upload

File: robotics_lab1/urdf/robot2DoF.urdf (robot description, URDF)
Before this commit: robot robot2DoF, 4 links, 3 joints
Joints:
- joint joint1: origin xyz=0 0 1.0 -> xyz=0 0 1.0 rpy=0 0 1.5708
- joint joint2: origin xyz=0.0 0.0 0.0 rpy=0 1.5708 0 -> xyz=0.0 -0.8 0.0 rpy=0 1.5708 -1.5708
